Commit message: Add differential drive and laser scan

File: my_rb1_description/urdf/my_rb1_robot.urdf (robot description, URDF)
Before this commit: robot my_rb1_robot, 7 links, 6 joints
Links:
- link front_laser: mass None -> 0.25; geometry collision sphere radius=0.01; visual sphere radius=0.01
Joints:
- joint base_link_base_footprint_joint: child base_link -> base_footprint; origin xyz=0 0 0.2 rpy=0 0 0 -> xyz=0 0 -0.2 rpy=0 0 0; parent base_footprint -> base_link

Commit message: Fix caster wheel position
Added a housing and located the origin of the caster wheel link at -15 cm from the base link

File: my_rb1_description/urdf/my_rb1_robot.urdf (robot description, URDF)
Before this commit: robot my_rb1_robot, 7 links, 6 joints
Links:
- link back_caster: mass 0.5 -> 1; geometry collision sphere radius=0.025; collision sphere radius=0.05
- link base_link: mass 22 -> 20
- link front_caster: mass 0.5 -> 1; geometry collision sphere radius=0.025; collision sphere radius=0.05
- link front_laser: mass 0.25 -> 1
Joints:
- joint back_caster_base_link_joint: origin xyz=-0.1 0.0 -0.175 rpy=0 0 0 -> xyz=-0.1 0.0 -0.15 rpy=0 0 0
- joint front_caster_base_link_joint: origin xyz=0.1 0.0 -0.175 rpy=0 0 0 -> xyz=0.1 0.0 -0.15 rpy=0 0 0

Commit message: Change caster wheel TF origin
The size of the housing was reduced

The TF of the caster wheels now matches their rotation axis

File: my_rb1_description/urdf/my_rb1_robot.urdf (robot description, URDF)
Before this commit: robot my_rb1_robot, 7 links, 6 joints
Links:
- link back_caster: geometry collision sphere radius=0.025; collision sphere radius=0.03
- link front_caster: geometry collision sphere radius=0.025; collision sphere radius=0.03
Joints:
- joint back_caster_base_link_joint: origin xyz=-0.1 0.0 -0.15 rpy=0 0 0 -> xyz=-0.1 0.0 -0.175 rpy=0 0 0
- joint front_caster_base_link_joint: origin xyz=0.1 0.0 -0.15 rpy=0 0 0 -> xyz=0.1 0.0 -0.175 rpy=0 0 0
